Commit message: arms.urdf is complete

File: urdf/arms.urdf (robot description, URDF)
Before this commit: robot arms, 5 links, 4 joints
Links:
- removed link body
- added link base_link; visual box size=0.06 0.14 0.16
Joints:
- joint left_elbow: axis (none) -> 0 0 1; limit (none) -> lower=-0.6 upper=0.6 effort=1000.0 velocity=0.5; origin xyz=0 0 0 -> xyz=0.15 0 0; type fixed -> revolute
- joint left_shoulder: axis (none) -> 0 0 1; limit (none) -> lower=-0.6 upper=0.6 effort=1000.0 velocity=0.5; origin xyz=0 0 0 -> xyz=0 0.07 0; parent body -> base_link; type fixed -> revolute
- joint right_elbow: axis (none) -> 0 0 1; limit (none) -> lower=-0.6 upper=0.6 effort=1000.0 velocity=0.5; origin xyz=0 0 0 -> xyz=0.15 0 0; type fixed -> revolute
- joint right_shoulder: axis (none) -> 0 0 1; limit (none) -> lower=-0.6 upper=0.6 effort=1000.0 velocity=0.5; origin xyz=0 0 0 -> xyz=0 -0.07 0; parent body -> base_link; type fixed -> revolute
