Commit message: Updated college.urdf origin

File: ros/src/colleague_description/urdf/colleague.urdf (robot description, URDF)
Before this commit: robot arms, 11 links, 10 joints
Joints:
- joint left_elbow: origin xyz=0.15 0 0 -> xyz=0.15 0 0 rpy=0 0 0
- joint left_finger_joint: origin xyz=0.03 0.015 0 -> xyz=0.03 0.015 0 rpy=0 0 0
- joint left_shoulder: origin xyz=0 0.07 0 -> xyz=0 0.07 0 rpy=0 0 0
- joint left_thumb_joint: origin xyz=0.03 -0.015 0 -> xyz=0.03 -0.015 0 rpy=0 0 0
- joint left_wrist_joint: origin xyz=0.15 0 0 -> xyz=0.15 0 0 rpy=0 0 0
- joint right_elbow: origin xyz=0.15 0 0 -> xyz=0.15 0 0 rpy=0 0 0
- joint right_finger_joint: origin xyz=0.03 -0.015 0 -> xyz=0.03 -0.015 0 rpy=0 0 0
- joint right_shoulder: origin xyz=0 -0.07 0 -> xyz=0 -0.07 0 rpy=0 0 0
- joint right_thumb_joint: origin xyz=0.03 0 0 -> xyz=0.03 0 0 rpy=0 0 0
- joint right_wrist_joint: origin xyz=0.15 0 0 -> xyz=0.15 0 0 rpy=0 0 0
